Commit message: fertiger brokk (testurdf) + erste brokk gazebo unternehmungen

File: description/brokk_v1_gazebo.xacro (robot description, xacro)
@@ -1,4 +1,4 @@
 <?xml version="1.0"?>
-<robot name="brokk_v1" xmlns:xacro="http://ros.org/wiki/xacro">
+<robot name="testurdf" xmlns:xacro="http://ros.org/wiki/xacro">
   <xacro:arg name="laser_visual"  default="false"/>
   <xacro:arg name="camera_visual" default="false"/>
@@ -17,4 +17,34 @@
     <material>Gazebo/FlatBlack</material>
   </gazebo>
+    <gazebo reference="wheel_left_mittelvorne_link">
+    <mu1>0.1</mu1>
+    <mu2>0.1</mu2>
+    <kp>500000.0</kp>
+    <kd>10.0</kd>
+    <minDepth>0.001</minDepth>
+    <maxVel>0.1</maxVel>
+    <fdir1>1 0 0</fdir1>
+    <material>Gazebo/FlatBlack</material>
+  </gazebo>
+    <gazebo reference="wheel_left_mittelhinten_link">
+    <mu1>0.1</mu1>
+    <mu2>0.1</mu2>
+    <kp>500000.0</kp>
+    <kd>10.0</kd>
+    <minDepth>0.001</minDepth>
+    <maxVel>0.1</maxVel>
+    <fdir1>1 0 0</fdir1>
+    <material>Gazebo/FlatBlack</material>
+  </gazebo>
+    <gazebo reference="wheel_left_behind_link">
+    <mu1>0.1</mu1>
+    <mu2>0.1</mu2>
+    <kp>500000.0</kp>
+    <kd>10.0</kd>
+    <minDepth>0.001</minDepth>
+    <maxVel>0.1</maxVel>
+    <fdir1>1 0 0</fdir1>
+    <material>Gazebo/FlatBlack</material>
+  </gazebo>
   <gazebo reference="wheel_right_link">
     <mu1>0.1</mu1>
@@ -27,20 +57,32 @@
     <material>Gazebo/FlatBlack</material>
   </gazebo>
-  <gazebo reference="caster_back_right_link">
-    <mu1>0.1</mu1>
-    <mu2>0.1</mu2>
-    <kp>1000000.0</kp>
-    <kd>100.0</kd>
-    <minDepth>0.001</minDepth>
-    <maxVel>1.0</maxVel>
-    <material>Gazebo/FlatBlack</material>
-  </gazebo>
-  <gazebo reference="caster_back_left_link">
-    <mu1>0.1</mu1>
-    <mu2>0.1</mu2>
-    <kp>1000000.0</kp>
-    <kd>100.0</kd>
-    <minDepth>0.001</minDepth>
-    <maxVel>1.0</maxVel>
+  <gazebo reference="wheel_right_mittelvorne_link">
+    <mu1>0.1</mu1>
+    <mu2>0.1</mu2>
+    <kp>500000.0</kp>
+    <kd>10.0</kd>
+    <minDepth>0.001</minDepth>
+    <maxVel>0.1</maxVel>
+    <fdir1>1 0 0</fdir1>
+    <material>Gazebo/FlatBlack</material>
+  </gazebo>
+  <gazebo reference="wheel_right_mittelhinten_link">
+    <mu1>0.1</mu1>
+    <mu2>0.1</mu2>
+    <kp>500000.0</kp>
+    <kd>10.0</kd>
+    <minDepth>0.001</minDepth>
+    <maxVel>0.1</maxVel>
+    <fdir1>1 0 0</fdir1>
+    <material>Gazebo/FlatBlack</material>
+  </gazebo>
+  <gazebo reference="wheel_right_behind_link">
+    <mu1>0.1</mu1>
+    <mu2>0.1</mu2>
+    <kp>500000.0</kp>
+    <kd>10.0</kd>
+    <minDepth>0.001</minDepth>
+    <maxVel>0.1</maxVel>
+    <fdir1>1 0 0</fdir1>
     <material>Gazebo/FlatBlack</material>
   </gazebo>
@@ -68,5 +110,5 @@
       <rightJoint>wheel_right_joint</rightJoint>
       <wheelSeparation>0.287</wheelSeparation>
-      <wheelDiameter>0.066</wheelDiameter>
+      <wheelDiameter>0.36</wheelDiameter>
       <wheelAcceleration>1</wheelAcceleration>
       <wheelTorque>10</wheelTorque>

File: description/testurdf.urdf.xacro (robot description, xacro)
@@ -2,5 +2,5 @@
 <robot name="testurdf" xmlns:xacro="http://ros.org/wiki/xacro">
   <xacro:include filename="$(find brokk)/description/common_properties.xacro"/>
-  <xacro:include filename="$(find brokk)/description/brokk_v1_gazebo.xacro"/>
+  <xacro:include filename="$(find brokk)/description/brokk_gazebo.xacro"/>
   <xacro:property name="joint_damping" value="100"/>
   <xacro:property name="PI" value="3.1415926535897931"/>
@@ -51,5 +51,5 @@
           <origin xyz="0.05 0 0" rpy="0 0 0" />
           <geometry>
-              <mesh filename="package://brokk/description/legs_final2.dae" />
+              <mesh filename="package://brokk/description/brokk_base_edit.stl" scale="0.011 0.01 0.01"/>
           </geometry>
           <material name="LightGrey">
@@ -60,5 +60,5 @@
           <origin xyz="-0.064 0 0.047" rpy="0 0 0"/>
           <geometry>
-              <mesh scale="0.0011 0.001 0.001" filename="package://brokk/description/legs.stl" />
+     	       <mesh filename="package://brokk/description/brokk_base_collision.stl"/> <!--1.725 0.52 0.6-->
           </geometry>
       </collision>
@@ -82,5 +82,5 @@
   <link name="brokk_base_structure">
       <visual>
-          <origin xyz="0.0 0.0 0.59 " rpy="0 0 0" />
+          <origin xyz="0.0 0.0 0.0" rpy="0 0 0" />
           <geometry>
               <mesh filename="package://brokk/description/base_final2.dae" />
@@ -105,5 +105,5 @@
     <parent link="base_link" />
     <child link = "brokk_base_structure" />
-    <origin xyz="0.0 0.0 0.0" rpy="0.0 0.0 1.57" />
+    <origin xyz="0.0 0.0 0.54" rpy="0.0 0.0 1.57" />
     <axis xyz="0 0 -1" />
     <limit effort="100.0" lower="${brokk_base_lower_limit}" upper="${brokk_base_upper_limit}" velocity="${brokk_arm_vel_limit}"/>
@@ -234,33 +234,235 @@
     </joint>
         <!-- brokk tip link ___________________________________________________________________________________________________________ -->
-    <link name="brokk_tip">
-        <visual>
-            <geometry>
-                <mesh scale="0.01 0.01 0.01" filename="package://brokk/description/tip.STL" />
-            </geometry>
-            <material name="LightGrey">
-                <color rgba="0.7 0.7 0.7 1.0"/>
-            </material>
-        </visual>
-        <collision>
-            <origin xyz="0 0 0" rpy="0 0 0" />
-            <geometry>
-                <mesh scale="0.01 0.01 0.01" filename="package://brokk/description/tip.STL" />
-            </geometry>
-        </collision>
-        <inertial>
-            <origin xyz="0 0 0" rpy="0 0 0" />
-            <mass value="2.34"/>
-            <inertia ixx="1.0" ixy="0.0" ixz="0.0" iyy="1.0" iyz="0.0" izz="1.0" />
-        </inertial>
-    </link>
-    <!--tip joint _________________________________________________________________________________________________________________ -->
-    <joint name="brokk_tip_jnt" type="fixed">
-      <parent link="brokk_arm4" />
-      <child link ="brokk_tip" />
-      <origin xyz="1.25 0 0.08" rpy="0.0 0.0 0.0" />
-      <axis xyz="0 1 0" />
-      <limit effort="0" lower="0" upper="0" velocity="0"/>
-      <dynamics damping="${joint_damping}"/>
-    </joint>
+  <!-- linker hinterer Reifen l0oo-->
+  <joint name="wheel_left_behind_joint" type="continuous">
+    <parent link="base_link"/>
+    <child link="wheel_left_behind_link"/>
+    <origin xyz="-0.46 0.40 0.18" rpy="0 0 0"/>
+    <axis xyz="0 1 0"/>
+  </joint>
+  <link name="wheel_left_behind_link">
+    <visual>
+      <origin xyz="0.0 0.0 0.0" rpy="1.57 0 0"/>
+      <geometry>
+     	 <cylinder radius="0.18" length="0.20"/>
+      </geometry>
+      <material name="green"/>
+    </visual>
+    <collision>
+      <origin xyz="0 0 0.0" rpy="1.57 0 0"/>
+      <geometry>
+        <cylinder length="0.2" radius="0.18"/>
+      </geometry>
+    </collision>
+    <inertial>
+      <origin xyz="0 0 0.0" />
+      <mass value="2.8498940e-02" />
+      <inertia ixx="1.1175580e-05" ixy="-4.2369783e-11" ixz="-5.9381719e-09"
+               iyy="1.1192413e-05" iyz="-1.4400107e-11"
+               izz="2.0712558e-05" />
+      </inertial>
+  </link>
+	<!-- linker mittel hinten Reifen loo0o-->
+  <joint name="wheel_left_mittelhinten_joint" type="continuous">
+    <parent link="base_link"/>
+    <child link="wheel_left_mittelhinten_link"/>
+    <origin xyz="-0.09 0.40 0.18" rpy="0 0 0"/>
+    <axis xyz="0 1 0"/>
+  </joint>
+  <link name="wheel_left_mittelhinten_link">
+    <visual>
+      <origin xyz="0.0 0.0 0.0" rpy="1.57 0 0"/>
+      <geometry>
+     	 <cylinder radius="0.18" length="0.20"/>
+      </geometry>
+      <material name="dark"/>
+    </visual>
+    <collision>
+      <origin xyz="0.0 0 0.0" rpy="1.57 0 0"/>
+      <geometry>
+        <cylinder length="0.2" radius="0.18"/>
+      </geometry>
+    </collision>
+    <inertial>
+      <origin xyz="0.0 0 0.0" />
+      <mass value="2.8498940e-02" />
+      <inertia ixx="1.1175580e-05" ixy="-4.2369783e-11" ixz="-5.9381719e-09"
+               iyy="1.1192413e-05" iyz="-1.4400107e-11"
+               izz="2.0712558e-05" />
+      </inertial>
+  </link>
+	<!-- linker mittel vorne Reifen lo0oo-->
+  <joint name="wheel__left_mittelvorne_joint" type="continuous">
+    <parent link="base_link"/>
+    <child link="wheel_left_mittelvorne_link"/>
+    <origin xyz="0.28 0.4 0.18" rpy="0 0 0"/>
+    <axis xyz="0 1 0"/>
+  </joint>
+  <link name="wheel_left_mittelvorne_link">
+    <visual>
+      <origin xyz="0 0 0" rpy="1.57 0 0"/>
+      <geometry>
+     	 <cylinder radius="0.18" length="0.2"/>
+      </geometry>
+      <material name="dark"/>
+    </visual>
+    <collision>
+      <origin xyz="0 0 0" rpy="1.57 0 0"/>
+      <geometry>
+        <cylinder length="0.2" radius="0.18"/>
+      </geometry>
+    </collision>
+    <inertial>
+      <origin xyz="0 0 0" />
+      <mass value="2.8498940e-02" />
+      <inertia ixx="1.1175580e-05" ixy="-4.2369783e-11" ixz="-5.9381719e-09"
+               iyy="1.1192413e-05" iyz="-1.4400107e-11"
+               izz="2.0712558e-05" />
+      </inertial>
+  </link>
+	<!-- rechter mittel hinten Reifen roo0o-->
+  <joint name="wheel_right_mittelhinten_joint" type="continuous">
+    <parent link="base_link"/>
+    <child link="wheel_right_mittelhinten_link"/>
+    <origin xyz="-0.08 -0.4 0.18" rpy="0 0 0"/>
+    <axis xyz="0 1 0"/>
+  </joint>
+  <link name="wheel_right_mittelhinten_link">
+    <visual>
+      <origin xyz="0.0 0 0.0" rpy="-1.57 0 0"/>
+      <geometry>
+      	<cylinder radius="0.18" length="0.2"/>
+      </geometry>
+      <material name="dark"/>
+    </visual>
+    <collision>
+      <origin xyz="0.0 0 0.0" rpy="-1.57 0 0"/>
+      <geometry>
+      	<cylinder radius="0.18" length="0.2"/>
+      </geometry>
+    </collision>
+    <inertial>
+      <origin xyz="0.0 0 0.0" />
+      <mass value="2.8498940e-02" />
+      <inertia ixx="1.1175580e-05" ixy="-4.2369783e-11" ixz="-5.9381719e-09"
+               iyy="1.1192413e-05" iyz="-1.4400107e-11"
+               izz="2.0712558e-05" />
+      </inertial>
+  </link>
+	<!-- rechter mittel vorne Reifen ro0oo-->
+  <joint name="wheel_right_mittelvorne_joint" type="continuous">
+    <parent link="base_link"/>
+    <child link="wheel_right_mittelvorne_link"/>
+    <origin xyz="0.28 -0.4 0.18" rpy="0 0 0"/>
+    <axis xyz="0 1 0"/>
+  </joint>
+  <link name="wheel_right_mittelvorne_link">
+    <visual>
+      <origin xyz="0 0 0.0" rpy="-1.57 0 0"/>
+      <geometry>
+      	<cylinder radius="0.18" length="0.2"/>
+      </geometry>
+      <material name="dark"/>
+    </visual>
+    <collision>
+      <origin xyz="0 0 0" rpy="-1.57 0 0"/>
+      <geometry>
+      	<cylinder radius="0.18" length="0.2"/>
+      </geometry>
+    </collision>
+    <inertial>
+      <origin xyz="0 0 0.0" />
+      <mass value="2.8498940e-02" />
+      <inertia ixx="1.1175580e-05" ixy="-4.2369783e-11" ixz="-5.9381719e-09"
+               iyy="1.1192413e-05" iyz="-1.4400107e-11"
+               izz="2.0712558e-05" />
+      </inertial>
+  </link>
+   <!-- linker vorderer Reifen looo0-->
+    <joint name="wheel_left_joint" type="continuous">
+    <parent link="base_link"/>
+    <child link="wheel_left_link"/>
+    <origin xyz="0.65 0.4 0.18" rpy="0 0 0"/>
+    <axis xyz="0 1 0"/>
+  </joint>
+  <link name="wheel_left_link">
+    <visual>
+      <origin xyz="0 0.0 0.0" rpy="1.57 0 0"/>
+      <geometry>
+      	<cylinder radius="0.18" length="0.2"/>
+      </geometry>
+      <material name="dark"/>
+    </visual>
+    <collision>
+      <origin xyz="0.0 0 0.0" rpy="1.57 0 0"/>
+      <geometry>
+        <cylinder length="0.2" radius="0.18"/>
+      </geometry>
+    </collision>
+    <inertial>
+      <origin xyz="0 0 0.0" />
+      <mass value="2.8498940e-02" />
+      <inertia ixx="1.1175580e-05" ixy="-4.2369783e-11" ixz="-5.9381719e-09"
+               iyy="1.1192413e-05" iyz="-1.4400107e-11"
+               izz="2.0712558e-05" />
+      </inertial>
+  </link>
+ <!-- rechter hinterer Reifen r0ooo -->
+  <joint name="wheel_right_behind_joint" type="continuous">
+    <parent link="base_link"/>
+    <child link="wheel_right_behind_link"/>
+    <origin xyz="-0.46 -0.4 0.18" rpy="0 0 0"/>
+    <axis xyz="0 1 0"/>
+  </joint>
+  <link name="wheel_right_behind_link">
+    <visual>
+      <origin xyz="0 0 0" rpy="-1.57 0 0"/>
+      <geometry>
+      	<cylinder radius="0.18" length="0.2"/>
+      </geometry>
+      <material name="blue"/>
+    </visual>
+    <collision>
+      <origin xyz="0 0 0.0" rpy="-1.57 0 0"/>
+      <geometry>
+      	<cylinder radius="0.18" length="0.2"/>
+      </geometry>
+    </collision>
+    <inertial>
+      <origin xyz="0 0 0.0" />
+      <mass value="2.8498940e-02" />
+      <inertia ixx="1.1175580e-05" ixy="-4.2369783e-11" ixz="-5.9381719e-09"
+               iyy="1.1192413e-05" iyz="-1.4400107e-11"
+               izz="2.0712558e-05" />
+      </inertial>
+  </link>
+   <!-- rechter vorderer Reifen rooo0-->
+    <joint name="wheel_right_joint" type="continuous">
+    <parent link="base_link"/>
+    <child link="wheel_right_link"/>
+    <origin xyz="0.65 -0.4 0.18" rpy="0 0 0"/>
+    <axis xyz="0 1 0"/>
+  </joint>
+  <link name="wheel_right_link">
+    <visual>
+      <origin xyz="0 0 0.0" rpy="-1.57 0 0"/>
+      <geometry>
+      	<cylinder radius="0.18" length="0.2"/>
+      </geometry>
+      <material name="dark"/>
+    </visual>
+    <collision>
+      <origin xyz="0 0 0.0" rpy="-1.57 0 0"/>
+      <geometry>
+      	<cylinder radius="0.18" length="0.2"/>
+      </geometry>
+    </collision>
+    <inertial>
+      <origin xyz="0 0 0.0" />
+      <mass value="2.8498940e-02" />
+      <inertia ixx="1.1175580e-05" ixy="-4.2369783e-11" ixz="-5.9381719e-09"
+               iyy="1.1192413e-05" iyz="-1.4400107e-11"
+               izz="2.0712558e-05" />
+      </inertial>
+  </link>
 </robot>
