Commit message: funktionierendes urdf

File: description/brokk_hishversion/brokk_vH.urdf.xacro (robot description, xacro)
@@ -71,2 +71,159 @@
       <dynamics damping="${joint_damping}"/>
     </joint>
+    <!-- also not sure which link _______________________________________________________________________________ -->
+    <link name="brokk_body1">
+        <visual>
+            <geometry>
+            <mesh  filename="package://brokk/description/brokk_hishversion/meshfiles/body1.dae"  />
+            </geometry>
+            <material name="LightGrey">
+            <color rgba="0.7 0.7 0.7 1.0"/>
+            </material>
+        </visual>
+        <collision>
+        <origin xyz="0 0 0" rpy="0 0 0" />
+            <geometry>
+            <mesh scale="0.001 0.001 0.001" filename="package://brokk/description/brokk_hishversion/meshfiles/body1.stl" />
+            </geometry>
+        </collision>
+        <inertial>
+            <origin xyz="0 0 0" rpy="0 0 0" />
+            <mass value="2.34"/>
+            <inertia ixx="1.0" ixy="0.0" ixz="0.0" iyy="1.0" iyz="0.0" izz="1.0" />
+        </inertial>
+    </link>
+    <!--body1 joint _______________________________________________________________________________________________ -->
+    <joint name="brokk_jnt1" type="revolute">
+        <parent link="$brokk_base" />
+        <child link = "brokk_body1" />
+        <origin xyz="0.493 0 0.078" rpy="0.0 -0.806 0.0" />
+        <axis xyz="0 1 0" />
+        <limit effort="100.0" lower="${brokk_body1_lower_limit}" upper="${brokk_body1_upper_limit}" velocity="${brokk_arm_vel_limit}"/>
+        <dynamics damping="${joint_damping}"/>
+    </joint>
+    <!--body2 link ________________________________________________________________________________________________ -->
+    <link name="brokk_body2">
+        <visual>
+            <geometry>
+                <mesh filename="package://brokk/description/brokk_hishversion/meshfiles/body2.dae" />
+            </geometry>
+            <material name="LightGrey">
+                <color rgba="0.7 0.7 0.7 1.0"/>
+            </material>
+        </visual>
+        <collision>
+	        <origin xyz="0 0 0" rpy="0 0 0" />
+            <geometry>
+                <mesh scale="0.001 0.001 0.001" filename="package://brokk/description/brokk_hishversion/meshfiles/body2.stl" />
+            </geometry>
+        </collision>
+        <inertial>
+            <origin xyz="0 0 0" rpy="0 0 0" />
+            <mass value="2.34"/>
+            <inertia ixx="1.0" ixy="0.0" ixz="0.0" iyy="1.0" iyz="0.0" izz="1.0" />
+        </inertial>
+    </link>
+    <!--body2 joint _________________________________________________________________________________________________ -->
+    <joint name="brokk_jnt2" type="revolute">
+      <parent link="brokk_body1" />
+      <child link ="brokk_body2" />
+      <origin xyz="0 0 0.87" rpy="0.0 0.78 0.0" />
+      <axis xyz="0 -1 0" />
+      <limit effort="100.0" lower="${brokk_body2_lower_limit }" upper="${brokk_body2_upper_limit }" velocity="0.5"/>
+      <dynamics damping="${joint_damping}"/>
+    </joint>
+    <!--body3 link __________________________________________________________________________________________________ -->
+    <link name="${prefix}brokk_body3">
+        <visual>
+            <geometry>
+                <mesh  filename="package://brokk/description/brokk_hishversion/meshfiles/body3.dae" />
+            </geometry>
+            <material name="LightGrey">
+                <color rgba="0.7 0.7 0.7 1.0"/>
+            </material>
+        </visual>
+        <collision>
+            <origin xyz="0 0 0" rpy="0 0 0" />
+            <geometry>
+                <mesh scale="0.001 0.001 0.001" filename="package://brokk/description/brokk_hishversion/meshfiles/body3.stl" />
+            </geometry>
+        </collision>
+        <inertial>
+            <origin xyz="0 0 0" rpy="0 0 0" />
+            <mass value="2.34"/>
+            <inertia ixx="1.0" ixy="0.0" ixz="0.0" iyy="1.0" iyz="0.0" izz="1.0" />
+        </inertial>
+    </link>
+    <!--body3 joint  __________________________________________________________________________________________________ -->
+    <joint name="$brokk_jnt3" type="revolute">
+        <parent link="brokk_body2" />
+        <child link ="brokk_body3" />
+        <origin xyz="1.37 0.0 0.01" rpy="0.0 1.75 0.0" />
+        <axis xyz="0 -1 0" />
+        <limit effort="100.0" lower="${brokk_body3_lower_limit }" upper="${brokk_body3_upper_limit }" velocity="0.5"/>
+        <dynamics damping="${joint_damping}"/>
+    </joint>
+    <!--body4 link _____________________________________________________________________________________________________ -->
+    <link name="$brokk_body4">
+        <visual>
+            <geometry>
+                <mesh  filename="package://brokk/description/brokk_hishversion/meshfiles/body4.dae"/>
+            </geometry>
+            <material name="LightGrey">
+                <color rgba="0.7 0.7 0.7 1.0"/>
+            </material>
+        </visual>
+        <collision>
+	        <origin xyz=" 0 0 0" rpy="0 0 0" />
+            <geometry>
+                <mesh scale="0.001 0.001 0.001" filename="package://brokk/description/brokk_hishversion/meshfiles/body4.stl" />
+            </geometry>
+        </collision>
+        <inertial>
+            <origin xyz="0 0 0" rpy="0 0 0" />
+            <mass value="2.34"/>
+            <inertia ixx="1.0" ixy="0.0" ixz="0.0" iyy="1.0" iyz="0.0" izz="1.0" />
+        </inertial>
+    </link>
+    <!--joint of body4___________________________________________________________________________________________________________ -->
+    <joint name="brokk_jnt4" type="revolute">
+      <parent link="brokk_body3" />
+      <child link ="brokk_body4" />
+      <origin xyz="0.89 0 0.0" rpy="0.0 -1.19 0.0" />
+      <axis xyz="0 1 0" />
+      <limit effort="100.0" lower="${brokk_body4_lower_limit }" upper="${brokk_body4_upper_limit }" velocity="2"/>
+     <dynamics damping="${joint_damping}"/>
+    </joint>
+    <!-- brokk tip link ___________________________________________________________________________________________________________ -->
+    <link name="brokk_tip">
+        <visual>
+            <geometry>
+                <mesh scale="0.01 0.01 0.01" filename="package://brokk/description/brokk_hishversion/meshfiles/tip.STL" />
+            </geometry>
+            <material name="LightGrey">
+                <color rgba="0.7 0.7 0.7 1.0"/>
+            </material>
+        </visual>
+        <collision>
+            <origin xyz="0 0 0" rpy="0 0 0" />
+            <geometry>
+                <mesh scale="0.01 0.01 0.01" filename="package://brokk/description/brokk_hishversion/meshfiles/tip.STL" />
+            </geometry>
+        </collision>
+        <inertial>
+            <origin xyz="0 0 0" rpy="0 0 0" />
+            <mass value="2.34"/>
+            <inertia ixx="1.0" ixy="0.0" ixz="0.0" iyy="1.0" iyz="0.0" izz="1.0" />
+        </inertial>
+    </link>
+    <!--tip joint _________________________________________________________________________________________________________________ -->
+    <joint name="$brokk_jnt5" type="fixed">
+      <parent link="brokk_body4" />
+      <child link ="brokk_tip" />
+      <origin xyz="1.25 0 0.08" rpy="0.0 0.0 0.0" />
+      <axis xyz="0 1 0" />
+      <limit effort="0" lower="0" upper="0" velocity="0"/>
+      <dynamics damping="${joint_damping}"/>
+    </joint>
+  </xacro:macro>
+</robot>
